Commit message: updates for openni2 deb package

File: asus_xtion_description/robots/asus_xtion.urdf.xacro (robot description, xacro)
@@ -1,14 +1,30 @@
 <?xml version="1.0" ?>
 <!-- Copyright (C) 2023  Miguel Ángel González Santamarta
-This program is free software: you can redistribute it and/or modify
-it under the terms of the GNU General Public License as published by
-the Free Software Foundation, either version 3 of the License, or
-(at your option) any later version.
-This program is distributed in the hope that it will be useful,
-but WITHOUT ANY WARRANTY; without even the implied warranty of
-MERCHANTABILITY or FITNESS FOR A PARTICULAR PURPOSE.  See the
-GNU General Public License for more details.
-You should have received a copy of the GNU General Public License
-along with this program.  If not, see <https://www.gnu.org/licenses/>. -->
+All rights reserved.
+Software License Agreement (BSD License 2.0)
+Redistribution and use in source and binary forms, with or without
+modification, are permitted provided that the following conditions
+are met:
+ * Redistributions of source code must retain the above copyright
+   notice, this list of conditions and the following disclaimer.
+ * Redistributions in binary form must reproduce the above
+   copyright notice, this list of conditions and the following
+   disclaimer in the documentation and/or other materials provided
+   with the distribution.
+ * Neither the name of the copyright holder nor the names of its
+   contributors may be used to endorse or promote products derived
+   from this software without specific prior written permission.
+THIS SOFTWARE IS PROVIDED BY THE COPYRIGHT HOLDERS AND CONTRIBUTORS
+"AS IS" AND ANY EXPRESS OR IMPLIED WARRANTIES, INCLUDING, BUT NOT
+LIMITED TO, THE IMPLIED WARRANTIES OF MERCHANTABILITY AND FITNESS
+FOR A PARTICULAR PURPOSE ARE DISCLAIMED. IN NO EVENT SHALL THE
+COPYRIGHT OWNER OR CONTRIBUTORS BE LIABLE FOR ANY DIRECT, INDIRECT,
+INCIDENTAL, SPECIAL, EXEMPLARY, OR CONSEQUENTIAL DAMAGES (INCLUDING,
+BUT NOT LIMITED TO, PROCUREMENT OF SUBSTITUTE GOODS OR SERVICES;
+LOSS OF USE, DATA, OR PROFITS; OR BUSINESS INTERRUPTION) HOWEVER
+CAUSED AND ON ANY THEORY OF LIABILITY, WHETHER IN CONTRACT, STRICT
+LIABILITY, OR TORT (INCLUDING NEGLIGENCE OR OTHERWISE) ARISING IN
+ANY WAY OUT OF THE USE OF THIS SOFTWARE, EVEN IF ADVISED OF THE
+POSSIBILITY OF SUCH DAMAGE. -->
 <robot name="asus_xtion" xmlns:xacro="http://www.ros.org/wiki/xacro">
     <!-- Include macros -->
@@ -17,5 +33,5 @@
     <link name="base_link"/>
     <!-- camera -->
-    <xacro:sensor_asus_xtion parent="base_link" name="openni">
+    <xacro:sensor_asus_xtion parent="base_link" name="camera">
         <origin xyz="0.0 0.0 0.0" rpy="0.0 0.0 0.0"/>
     </xacro:sensor_asus_xtion>

File: asus_xtion_description/urdf/asus_xtion.urdf.xacro (robot description, xacro)
@@ -1,26 +1,81 @@
 <?xml version="1.0"?>
 <!-- Copyright (C) 2023  Miguel Ángel González Santamarta
-This program is free software: you can redistribute it and/or modify
-it under the terms of the GNU General Public License as published by
-the Free Software Foundation, either version 3 of the License, or
-(at your option) any later version.
-This program is distributed in the hope that it will be useful,
-but WITHOUT ANY WARRANTY; without even the implied warranty of
-MERCHANTABILITY or FITNESS FOR A PARTICULAR PURPOSE.  See the
-GNU General Public License for more details.
-You should have received a copy of the GNU General Public License
-along with this program.  If not, see <https://www.gnu.org/licenses/>. -->
+All rights reserved.
+Software License Agreement (BSD License 2.0)
+Redistribution and use in source and binary forms, with or without
+modification, are permitted provided that the following conditions
+are met:
+ * Redistributions of source code must retain the above copyright
+   notice, this list of conditions and the following disclaimer.
+ * Redistributions in binary form must reproduce the above
+   copyright notice, this list of conditions and the following
+   disclaimer in the documentation and/or other materials provided
+   with the distribution.
+ * Neither the name of the copyright holder nor the names of its
+   contributors may be used to endorse or promote products derived
+   from this software without specific prior written permission.
+THIS SOFTWARE IS PROVIDED BY THE COPYRIGHT HOLDERS AND CONTRIBUTORS
+"AS IS" AND ANY EXPRESS OR IMPLIED WARRANTIES, INCLUDING, BUT NOT
+LIMITED TO, THE IMPLIED WARRANTIES OF MERCHANTABILITY AND FITNESS
+FOR A PARTICULAR PURPOSE ARE DISCLAIMED. IN NO EVENT SHALL THE
+COPYRIGHT OWNER OR CONTRIBUTORS BE LIABLE FOR ANY DIRECT, INDIRECT,
+INCIDENTAL, SPECIAL, EXEMPLARY, OR CONSEQUENTIAL DAMAGES (INCLUDING,
+BUT NOT LIMITED TO, PROCUREMENT OF SUBSTITUTE GOODS OR SERVICES;
+LOSS OF USE, DATA, OR PROFITS; OR BUSINESS INTERRUPTION) HOWEVER
+CAUSED AND ON ANY THEORY OF LIABILITY, WHETHER IN CONTRACT, STRICT
+LIABILITY, OR TORT (INCLUDING NEGLIGENCE OR OTHERWISE) ARISING IN
+ANY WAY OUT OF THE USE OF THIS SOFTWARE, EVEN IF ADVISED OF THE
+POSSIBILITY OF SUCH DAMAGE. -->
 <robot name="sensor_asus_xtion" xmlns:xacro="http://www.ros.org/wiki/xacro">
   <xacro:macro name="sensor_asus_xtion" params="name parent *origin ">
     <xacro:property name="M_SCALE_XTION" value="0.001"/>
-    <xacro:property name="asus_xtion_pro_depth_rel_rgb_py" value="0.0270" />
-    <xacro:property name="asus_xtion_pro_cam_rel_rgb_py"   value="-0.0220" />
     <xacro:property name="M_PI" value="3.1415926535897931" />
-    <joint name="${name}_cam_rgb_joint" type="fixed">
+    <link name="${name}_link">
+      <visual>
+        <origin xyz="0 0 0" rpy="${-M_PI/2} -${M_PI} ${-M_PI/2}"/>
+        <geometry>
+          <mesh filename="package://asus_xtion_description/meshes/asus_xtion_pro_live.dae" scale="${M_SCALE_XTION} ${M_SCALE_XTION} ${M_SCALE_XTION}"/>
+        </geometry>
+      </visual>
+      <!--collision>
+        <origin xyz="0.0 0.0 0.0" rpy="0 0 0" />
+        <geometry>
+          <box size="0.0730 .2760 0.0720"/>
+        </geometry>
+      </collision-->
+      <collision>
+        <origin xyz="0 0 0" rpy="${-M_PI/2} -${M_PI} ${-M_PI/2}"/>
+        <geometry>
+          <mesh filename="package://asus_xtion_description/meshes/asus_xtion_pro_live.dae" scale="${M_SCALE_XTION} ${M_SCALE_XTION} ${M_SCALE_XTION}"/>
+        </geometry>
+      </collision>
+      <inertial>
+        <mass value="0.01" />
+        <origin xyz="0 0 0" />
+        <inertia ixx="0.001" ixy="0.0" ixz="0.0"
+          iyy="0.001" iyz="0.0"
+          izz="0.001" />
+      </inertial>
+    </link>
+    <joint name="${name}_camera_joint" type="fixed">
 	  <xacro:insert_block name="origin" />
       <parent link="${parent}"/>
+      <child link="${name}_link" />
+    </joint>
+    <link name="${name}_rgb_frame">
+      <inertial>
+        <mass value="0.001" />
+        <origin xyz="0 0 0" />
+        <inertia ixx="0.001" ixy="0.0" ixz="0.0"
+          iyy="0.001" iyz="0.0"
+          izz="0.001" />
+      </inertial>
+    </link>
+    <joint name="${name}_rgb_joint" type="fixed">
+      <origin xyz="0 0.022 0" rpy="0 0 0"/>
+      <parent link="${name}_link" />
       <child link="${name}_rgb_frame" />
     </joint>
-    <link name="${name}_rgb_frame">
+    <link name="${name}_rgb_optical_frame">
       <inertial>
         <mass value="0.001" />
@@ -36,38 +91,5 @@
       <child link="${name}_rgb_optical_frame" />
     </joint>
-    <link name="${name}_rgb_optical_frame">
-      <inertial>
-        <mass value="0.001" />
-        <origin xyz="0 0 0" />
-        <inertia ixx="0.001" ixy="0.0" ixz="0.0"
-          iyy="0.001" iyz="0.0"
-          izz="0.001" />
-      </inertial>
-    </link>
-    <joint name="${name}_cam_joint" type="fixed">
-      <origin xyz="0 ${asus_xtion_pro_cam_rel_rgb_py} 0"
-              rpy="0 0 0"/>
-      <parent link="${name}_rgb_frame"/>
-      <child link="${name}_cam_link"/>
-    </joint>
-    <link name="${name}_cam_link">
-      <visual>
-        <origin xyz="-0.01 0.02 0" rpy="${-M_PI/2} -${M_PI} ${-M_PI/2}"/>
-        <geometry>
-          <mesh filename="package://asus_xtion_description/meshes/asus_xtion_pro_live.dae" scale="${M_SCALE_XTION} ${M_SCALE_XTION} ${M_SCALE_XTION}"/>
-        </geometry>
-      </visual>
-      <!--collision>
-        <origin xyz="0.0 0.0 0.0" rpy="0 0 0" />
-        <geometry>
-          <box size="0.0730 .2760 0.0720"/>
-        </geometry>
-      </collision-->
-      <collision>
-        <origin xyz="-0.01 0.02 0.0" rpy="${-M_PI/2} -${M_PI} ${-M_PI/2}" />
-        <geometry>
-          <mesh filename="package://asus_xtion_description/meshes/asus_xtion_pro_live.dae" scale="${M_SCALE_XTION} ${M_SCALE_XTION} ${M_SCALE_XTION}"/>
-        </geometry>
-      </collision>
+    <link name="${name}_depth_frame">
       <inertial>
         <mass value="0.01" />
@@ -79,21 +101,7 @@
     </link>
     <joint name="${name}_depth_joint" type="fixed">
-      <origin xyz="0 ${asus_xtion_pro_depth_rel_rgb_py} 0" rpy="0 0 0" />
-      <parent link="${name}_rgb_frame" />
+      <origin xyz="0 0.049 0" rpy="0 0 0" />
+      <parent link="${name}_link" />
       <child link="${name}_depth_frame" />
-    </joint>
-    <link name="${name}_depth_frame">
-      <inertial>
-        <mass value="0.01" />
-        <origin xyz="0 0 0" />
-        <inertia ixx="0.001" ixy="0.0" ixz="0.0"
-          iyy="0.001" iyz="0.0"
-          izz="0.001" />
-      </inertial>
-    </link>
-    <joint name="${name}_cam_depth_optical_joint" type="fixed">
-      <origin xyz="0 0 0" rpy="${-M_PI/2} 0 ${-M_PI/2}" />
-      <parent link="${name}_depth_frame" />
-      <child link="${name}_depth_optical_frame" />
     </joint>
     <link name="${name}_depth_optical_frame">
@@ -106,4 +114,9 @@
       </inertial>
     </link>
+    <joint name="${name}_depth_optical_joint" type="fixed">
+      <origin xyz="0 0 0" rpy="${-M_PI/2} 0 ${-M_PI/2}" />
+      <parent link="${name}_depth_frame" />
+      <child link="${name}_depth_optical_frame" />
+    </joint>
     <!-- gazebo plugin -->
     <gazebo reference="${name}_depth_frame">
@@ -113,13 +126,13 @@
         <visualize>false</visualize>
         <camera>
-          <horizontal_fov>1.57</horizontal_fov>
+          <horizontal_fov>${62.8 * M_PI/180.0}</horizontal_fov>
           <image>
-            <width>720</width>
+            <width>640</width>
             <height>480</height>
             <format>R8G8B8</format>
           </image>
           <clip>
-            <near>0.1</near>
-            <far>100</far>
+            <near>0.05</near>
+            <far>9</far>
           </clip>
           <noise>

Commit message: Renaming asus xtion camera to openni

File: asus_xtion_description/robots/asus_xtion.urdf.xacro (robot description, xacro)
@@ -28,11 +28,11 @@
 POSSIBILITY OF SUCH DAMAGE. -->
 <robot name="asus_xtion" xmlns:xacro="http://www.ros.org/wiki/xacro">
-    <!-- Include macros -->
-    <xacro:include filename="$(find asus_xtion_description)/urdf/asus_xtion.urdf.xacro"/>
-    <!-- The base link -->
-    <link name="base_link"/>
-    <!-- camera -->
-    <xacro:sensor_asus_xtion parent="base_link" name="camera">
-        <origin xyz="0.0 0.0 0.0" rpy="0.0 0.0 0.0"/>
-    </xacro:sensor_asus_xtion>
+  <!-- Include macros -->
+  <xacro:include filename="$(find asus_xtion_description)/urdf/asus_xtion.urdf.xacro"/>
+  <!-- The base link -->
+  <link name="base_link"/>
+  <!-- camera -->
+  <xacro:sensor_asus_xtion parent="base_link" name="openni">
+    <origin xyz="0.0 0.0 0.0" rpy="0.0 0.0 0.0"/>
+  </xacro:sensor_asus_xtion>
 </robot>
